Commit message: Fix camera adapter mounting and update README

File: xarm7_xhand_direct_camera.urdf (robot description, URDF)
Before this commit: robot xarm7_xhand_direct_camera, 30 links, 29 joints
Links:
- added link adapter_camera_link; collision mesh filename=meshes/adapter/xhand_adapter_camera.stl scale=0.001 0.001 0.001; visual mesh filename=meshes/adapter/xhand_adapter_camera.stl scale=0.001 0.001 0.001
- link link7: geometry collision mesh filename=meshes/xarm7_1305/collision/link7.obj; visual mesh filename=meshes/xarm7_1305/visual/link7.dae
Joints:
- removed joint right_hand_to_d405_camera_1
- removed joint right_hand_to_d405_camera_2
- added joint adapter_to_d405_camera_1: type fixed, parent adapter_camera_link, child d405_camera_1_link, origin xyz=0.0329323 0.00173235 0.0939772 rpy=2.6180357 1.1082600 -1.5707742
- added joint adapter_to_d405_camera_2: type fixed, parent adapter_camera_link, child d405_camera_2_link, origin xyz=-0.0608978 0.0349099 -0.0266976 rpy=-0.1305675 1.4785020 1.5705475
- added joint link7_to_adapter_camera: type fixed, parent link7, child adapter_camera_link, origin xyz=0 0 0.0005 rpy=1.5708 0 3.1416
- joint xhand_mount_joint: origin xyz=0 0 0.025 rpy=3.14159265 0 1.5707963 -> xyz=0 0.0245 0 rpy=-1.1086034 -1.5707881 2.6793997; parent link7 -> adapter_camera_link
