Commit message: Add virtual palm frames to Wuji assets and document RL integration

File: xarm7_wuji_90.urdf (robot description, URDF)
Before this commit: robot xarm7_wuji_90, 34 links, 33 joints
Links:
- added link palm_center
Joints:
- added joint palm_center_joint: type fixed, parent right_palm_link, child palm_center, origin xyz=0.004 -0.0023529 0.0434161 rpy=0 0 0

File: xarm7_wuji_90_camera.urdf (robot description, URDF)
Before this commit: robot xarm7_wuji_90_camera, 39 links, 38 joints
Links:
- added link palm_center
Joints:
- added joint palm_center_joint: type fixed, parent right_palm_link, child palm_center, origin xyz=0.004 -0.0023529 0.0434161 rpy=0 0 0

File: xarm7_wuji_direct.urdf (robot description, URDF)
Before this commit: robot xarm7_wuji_direct, 34 links, 33 joints
Links:
- added link palm_center
Joints:
- added joint palm_center_joint: type fixed, parent right_palm_link, child palm_center, origin xyz=0.004 -0.0023529 0.0434161 rpy=0 0 0

File: xarm7_wuji_direct_camera.urdf (robot description, URDF)
Before this commit: robot xarm7_wuji_direct_camera, 38 links, 37 joints
Links:
- added link palm_center
Joints:
- added joint palm_center_joint: type fixed, parent right_palm_link, child palm_center, origin xyz=0.004 -0.0023529 0.0434161 rpy=0 0 0
